File: dice-keychain/dice-keychain.kicad_sch (KiCad schematic)
At the start: 16 parts, among them J1 Conn_01x06_Pin, SW1 SW_Push_Dual, U1 ATtiny85-20S

Commit message: finished coding
Parts:
- R1, R2, R3, R4: value 1k -> 330
Changed lines of the file:
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@@
 			)
 		)
-		(property "Value" "1k"
+		(property "Value" "330"
 			(at 173.99 69.85 90)
 			(effects
@@
 			)
 		)
-		(property "Value" "1k"
+		(property "Value" "330"
 			(at 173.99 104.14 90)
 			(effects
@@
 			)
 		)
-		(property "Value" "1k"
+		(property "Value" "330"
 			(at 173.99 81.28 90)
 			(effects
@@
 			)
 		)
-		(property "Value" "1k"
+		(property "Value" "330"
 			(at 173.99 92.71 90)
 			(effects
